File: ergogen/output/pcbs/tutorial.kicad_pcb (KiCad board)
At the start: 2 copper layers, 275.3 x 146.2 mm, 74 parts

Commit message: feat: alpha4, proper scale
Parts:
- moved D36 111.3 mm to (126.6, 180.3), turned to 40 degrees
- moved S36 110.1 mm to (123.4, 176.4), turned to 40 degrees
- moved D1 102.0 mm to (33.6, 32.1), turned to -41 degrees
- moved S1 100.4 mm to (36.9, 28.4), turned to -41 degrees
- moved D35 96.7 mm to (147.2, 167.2), turned to 25 degrees
- moved S35 94.7 mm to (145.1, 162.6), turned to 25 degrees
- moved D34 87.6 mm to (165.2, 160.6), turned to 15 degrees
- moved B1 85.8 mm to (151.2, 122.6), turned to -25 degrees
- moved D17 85.3 mm to (238.9, 152.0), turned to -9 degrees
- moved S34 84.9 mm to (163.9, 155.8), turned to 15 degrees
- moved S17 83.3 mm to (239.6, 147.1), turned to -9 degrees
- moved D18 78.4 mm to (241.6, 134.7), turned to -9 degrees
- moved S18 76.5 mm to (242.4, 129.8), turned to -9 degrees
- moved D19 76.0 mm to (219.3, 136.3), turned to -3 degrees
- moved D28 75.3 mm to (163.9, 137.3), turned to 0 degrees
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Connections:
- net mirror_tucky_default renamed mirror_inner_default
- net tucky_default renamed inner_default
- D1 pad 1: P2 -> P0
- D1 pad 2: pinky_bottom -> pinky_extension_home
- D16 pad 1: P6 -> P4
- D16 pad 2: mirror_pinky_bottom -> mirror_pinky_extension_home
- D17 pad 1: P5 -> P6
- D17 pad 2: mirror_pinky_home -> mirror_pinky_bottom
- D18 pad 1: P4 -> P5
- D18 pad 2: mirror_pinky_top -> mirror_pinky_home
- D2 pad 1: P1 -> P2
- D2 pad 2: pinky_home -> pinky_bottom
- D3 pad 1: P0 -> P1
- D3 pad 2: pinky_top -> pinky_home
- S1 pad 2: pinky_bottom -> pinky_extension_home
- S16 pad 2: mirror_pinky_bottom -> mirror_pinky_extension_home
- S17 pad 2: mirror_pinky_home -> mirror_pinky_bottom
- S18 pad 2: mirror_pinky_top -> mirror_pinky_home
- S2 pad 2: pinky_home -> pinky_bottom
- S3 pad 2: pinky_top -> pinky_home
Other:
- board size 275.3 x 146.2 mm -> 251.2 x 177.2 mm
- net class Default removed

Commit message: feat: alpha 5, thumb update
Parts:
- moved D1 77.6 mm to (48.1, 108.4), turned to -18.5 degrees
- moved D2 77.2 mm to (60.1, 130.8), turned to -18.5 degrees
- moved D33 77.1 mm to (152.8, 201.3), turned to -67.5 degrees
- moved S1 76.3 mm to (49.7, 103.6), turned to -18.5 degrees
- moved S33 75.9 mm to (157.4, 199.4), turned to -67.5 degrees
- moved S2 75.7 mm to (61.7, 126.1), turned to -18.5 degrees
- moved D3 72.3 mm to (65.6, 114.2), turned to -18.5 degrees
- moved S3 70.9 mm to (67.2, 109.5), turned to -18.5 degrees
- moved D32 69.9 mm to (137.6, 181.6), turned to -37.5 degrees
- moved D36 69.6 mm to (192.9, 201.3), turned to 67.5 degrees
- moved S36 68.9 mm to (188.3, 199.4), turned to 67.5 degrees
- moved D31 68.5 mm to (122.2, 170.8), turned to -32.5 degrees
- moved D4 67.9 mm to (84.7, 125.9), turned to -24.5 degrees
- moved S32 66.8 mm to (140.7, 177.6), turned to -37.5 degrees
- moved S4 66.3 mm to (86.8, 121.3), turned to -24.5 degrees
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Other:
- board size 251.2 x 177.2 mm -> 273.7 x 139.1 mm
- net class Default added: clearance 0.2, trace_width 0.25, via_dia 0.8, via_drill 0.4

Commit message: feat: alpha 7, keys position final
Parts:
- added JST1: , JST_PH_S2B-PH-K_02x2.00mm_Angled, F.Cu at (183.5, 136.8)
- moved B1 9.27 mm to (184.5, 147.9)
- moved S31 8.53 mm to (116.6, 168.8), turned to -29 degrees
- moved D31 8.32 mm to (114.2, 173.1), turned to -29 degrees
- moved S33 8.10 mm to (149.8, 196.5), turned to -62 degrees
- moved D33 7.76 mm to (145.4, 198.8), turned to -62 degrees
- moved S32 7.73 mm to (133.0, 178.4), turned to -32 degrees
- moved D32 7.37 mm to (130.3, 182.6), turned to -32 degrees
- moved D13 6.19 mm to (129.0, 156.8), turned to -29 degrees
- moved S13 6.15 mm to (131.4, 152.4), turned to -29 degrees
- moved D14 6.08 mm to (137.5, 141.4), turned to -29 degrees
- moved S14 6.05 mm to (139.9, 137.1), turned to -29 degrees
- moved D15 5.99 mm to (146.0, 126.1), turned to -29 degrees
- moved S15 5.97 mm to (148.4, 121.8), turned to -29 degrees
- moved MCU1 5.91 mm to (169.5, 158.0)
- moved S30 5.84 mm to (190.6, 121.8), turned to 29 degrees
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Connections:
- D1 pad 1: P0 -> P3
- D10 pad 1: P2 -> P5
- D11 pad 1: P1 -> P4
- D12 pad 1: P0 -> P3
- D13 pad 1: P2 -> P5
- D14 pad 1: P1 -> P4
- D15 pad 1: P0 -> P3
- D16 pad 1: P4 -> P19
- D17 pad 1: P6 -> P15
- D18 pad 1: P5 -> P18
- D19 pad 1: P6 -> P15
- D2 pad 1: P2 -> P5
- D20 pad 1: P5 -> P18
- D21 pad 1: P4 -> P19
- D22 pad 1: P6 -> P15
- D23 pad 1: P5 -> P18
- D24 pad 1: P4 -> P19
- D25 pad 1: P6 -> P15
- D26 pad 1: P5 -> P18
- D27 pad 1: P4 -> P19
- D28 pad 1: P6 -> P15
- D29 pad 1: P5 -> P18
- D3 pad 1: P1 -> P4
- D30 pad 1: P4 -> P19
- D31 pad 1: P3 -> P6
- D32 pad 1: P3 -> P6
- D33 pad 1: P3 -> P6
- D34 pad 1: P7 -> P14
- D35 pad 1: P7 -> P14
- D36 pad 1: P7 -> P14
- D4 pad 1: P2 -> P5
- D5 pad 1: P1 -> P4
- D6 pad 1: P0 -> P3
- D7 pad 1: P2 -> P5
- D8 pad 1: P1 -> P4
- D9 pad 1: P0 -> P3
- S1 pad 1: P8 -> P7
- S10 pad 1: P14 -> P16
- S11 pad 1: P14 -> P16
- S12 pad 1: P14 -> P16
- S13 pad 1: P15 -> P10
- S14 pad 1: P15 -> P10
- S15 pad 1: P15 -> P10
- S16 pad 1: P8 -> P7
- S17 pad 1: P8 -> P7
- S18 pad 1: P8 -> P7
- S19 pad 1: P9 -> P8
- S2 pad 1: P8 -> P7
- S20 pad 1: P9 -> P8
- S21 pad 1: P9 -> P8
- S22 pad 1: P10 -> P9
- S23 pad 1: P10 -> P9
- S24 pad 1: P10 -> P9
- S25 pad 1: P14 -> P16
- S26 pad 1: P14 -> P16
- S27 pad 1: P14 -> P16
- S28 pad 1: P15 -> P10
- S29 pad 1: P15 -> P10
- S3 pad 1: P8 -> P7
- S30 pad 1: P15 -> P10
- S31 pad 1: P10 -> P9
- S32 pad 1: P14 -> P16
- S33 pad 1: P15 -> P10
- S34 pad 1: P10 -> P9
- S35 pad 1: P14 -> P16
- S36 pad 1: P15 -> P10
- S4 pad 1: P9 -> P8
- S5 pad 1: P9 -> P8
- S6 pad 1: P9 -> P8
- S7 pad 1: P10 -> P9
- S8 pad 1: P10 -> P9
- S9 pad 1: P10 -> P9
Other:
- board size 273.7 x 139.1 mm -> 272.7 x 132.7 mm
