File: pcb/tolkeeb_zero.kicad_pcb (KiCad board)
At the start: 2 copper layers, 242.8 x 178.3 mm, 115 parts

Commit message: chore: ?
Parts:
- moved D1 65.6 mm to (23.6, 122.5), turned to 160 degrees
- moved S1 65.0 mm to (25.2, 118.0), turned to -20 degrees
- moved SB1 65.0 mm to (25.2, 118.0), turned to -20 degrees
- moved D2 60.2 mm to (35.0, 145.2), turned to 160 degrees
- moved S2 59.2 mm to (36.6, 140.8), turned to -20 degrees
- moved SB2 59.2 mm to (36.6, 140.8), turned to -20 degrees
- moved D16 59.0 mm to (271.9, 122.5), turned to -160 degrees
- moved S16 58.4 mm to (270.3, 118.0), turned to 20 degrees
- moved SB16 58.4 mm to (270.3, 118.0), turned to 20 degrees
- moved D3 56.8 mm to (41.0, 128.8), turned to 160 degrees
- moved S3 56.1 mm to (42.6, 124.4), turned to -20 degrees
- moved SB3 56.1 mm to (42.6, 124.4), turned to -20 degrees
- moved D17 53.6 mm to (260.5, 145.2), turned to -160 degrees
- moved S17 52.6 mm to (258.9, 140.8), turned to 20 degrees
- moved SB17 52.6 mm to (258.9, 140.8), turned to 20 degrees
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Other:
- board size 242.8 x 178.3 mm -> 272.7 x 132.7 mm
