File: pcb/tolkeeb_zero.kicad_pcb (KiCad board)
At the start: 2 copper layers, 272.7 x 132.7 mm, 115 parts

Commit message: feat: full routing + silkscreen
Parts:
- added G***: LOGO, Tolki:tachikoma15, F.Cu at (150.6, 198.2)
- moved B1 56.6 mm to (158.5, 147.3)
- moved S4 6.72 mm to (64.1, 131.5)
- moved SB4 6.72 mm to (64.1, 131.5)
- moved D26 6.72 mm to (197.5, 137.4)
- moved D27 6.72 mm to (189.0, 122.1)
- moved D30 6.72 mm to (173.8, 132.9)
- moved D33 6.72 mm to (126.6, 205.6)
- moved D34 6.72 mm to (205.6, 179.8)
- moved D7 6.72 mm to (80.8, 139.8)
- moved JST1 6.72 mm to (150.4, 144.7)
- moved S17 6.72 mm to (261.6, 134.6)
- moved SB17 6.72 mm to (261.6, 134.6)
- moved D21 6.72 mm to (223.4, 104.2)
- moved S21 6.72 mm to (221.3, 100.0)
- moved S24 6.72 mm to (200.7, 105.1)
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Routing:
- net P7: track 73.6 -> 339.5 mm, vias 0 -> 1
- net P8: track 70.0 -> 288.9 mm, vias 0 -> 2
- net P19: track 0.00 -> 207.3 mm, vias 0 -> 4
- net P3: track 0.00 -> 194.2 mm, vias 0 -> 5
- net P15: track 0.00 -> 189.8 mm, vias 0 -> 4
- net P18: track 0.00 -> 185.5 mm, vias 0 -> 4
- net P9: track 163.8 -> 349.2 mm, vias 0 -> 3
- net P4: track 0.00 -> 156.6 mm, vias 0 -> 5
- net P5: track 0.00 -> 156.6 mm, vias 0 -> 5
- net P16: track 158.7 -> 302.7 mm, vias 0 -> 2
- net P10: track 171.3 -> 278.7 mm, vias 0 -> 2
- net P14: track 0.00 -> 75.3 mm, vias 0 -> 3
- net P6: track 0.00 -> 72.4 mm, vias 0 -> 3
- net GND: track 0.00 -> 32.5 mm
- net RAW: track 0.00 -> 14.9 mm
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